File: BSPD/BSPD.kicad_pcb (KiCad board)
At the start: 2 copper layers, 66 x 42 mm, 79 parts, among them J2 282834-6, K2 G5Q-1A, Q1 BSS84, Q2 MMBT2222A, Q3 MMBT2222A, U1 LM339, U2 LM339, U3 74LVC2G00, U4 74HC00, U5 74LVC2G04, U6 LM311, U7 LM555xM, U8 74AHC1G32, U9 AMS1117-5.0

Commit message: v1.1
Parts:
- removed U9: AMS1117-5.0, Package_TO_SOT_SMD:SOT-223-3_TabPin2
- added D8: SMF18A, Diode_SMD:D_SMF, F.Cu at (114.1, 105.8)
- added F1: 150mA, Fuse:Fuse_1812_4532Metric_Pad1.30x3.40mm_HandSolder, F.Cu at (120.6, 120.1)
- added VR1: TPS7B6950QDCYRQ1, TPS7B6950QDCYRQ1:VREG_TPS7B6950QDCYRQ1, F.Cu at (119.6, 111.6)
- H1, H2, H3, H4: footprint MountingHole:MountingHole_2.2mm_M2_Pad -> MountingHole:MountingHole_3.2mm_M3_Pad
- R23, R24, R25, R26, R27: value 220 -> 470
- U1, U2: footprint LM339:SOIC127P600X175-14N -> lm339:SOIC127P600X175-14N
- U3: footprint SN74LVC2G00DCUT:SOP50P310X90-8N -> SN74LVC2G00:SOP50P310X90-8N
- moved C16 4.32 mm to (113.4, 109.8)
- moved C1 4.32 mm to (114.6, 109.8)
- moved TP2 2.10 mm to (125.3, 87.8)
- moved C15 1.95 mm to (113.4, 113.4)
- moved C2 1.95 mm to (114.6, 113.4)
- moved TP1 1.89 mm to (120.9, 87.8)
- moved H1 0.89 mm to (114.5, 87.8)
- moved H2 0.89 mm to (114.5, 119.8)
- moved H3 0.89 mm to (170.5, 87.8)
- moved H4 0.89 mm to (170.5, 119.8)
Connections:
- C1 pad 1: +12V -> Net-(D8-A1)
- C16 pad 1: +12V -> Net-(D8-A1)
Routing:
- net Net-(D8-A1): track 0.00 -> 17.6 mm
- net +12V: track 22.8 -> 10.9 mm
- net +5V: track 42.7 -> 39.3 mm
- net Net-(U1A--): track 27.6 -> 26.8 mm
- net Net-(U2A--): track 18.7 -> 19.3 mm
- net GND: track 50.2 -> 50.7 mm, vias 39 -> 43
