File: BSPD/BSPD.kicad_sch (KiCad schematic)
At the start: 78 parts, among them J2 282834-6, K2 G5Q-1A, Q1 BSS84, Q2 MMBT2222A, Q3 MMBT2222A, U1 LM339, U2 LM339, U3 74LVC2G00, U4 74HC00, U5 74LVC2G04, U6 LM311, U7 LM555xM, U8 74AHC1G32, U9 AMS1117-5.0

Commit message: v1.1
Parts:
- removed U9: AMS1117-5.0, Package_TO_SOT_SMD:SOT-223-3_TabPin2, symbol Regulator_Linear:AMS1117-5.0
- added D8: SMF18A, Diode_SMD:D_SMF, symbol Diode:SMF18A
- added F1: 150mA, Fuse:Fuse_1812_4532Metric_Pad1.30x3.40mm_HandSolder, symbol Device:Fuse
- added VR1: TPS7B6950QDCYRQ1, TPS7B6950QDCYRQ1:VREG_TPS7B6950QDCYRQ1, symbol TPS7B6950QDCYRQ1:TPS7B6950QDCYRQ1
- H1, H2, H3, H4: footprint MountingHole:MountingHole_2.2mm_M2_Pad -> MountingHole:MountingHole_3.2mm_M3_Pad
- U1, U2: footprint LM339:SOIC127P600X175-14N -> lm339:SOIC127P600X175-14N
- U3: footprint SN74LVC2G00DCUT:SOP50P310X90-8N -> SN74LVC2G00:SOP50P310X90-8N
Connections:
- net +12V: now also F1.1; no longer C1.1, C16.1
- net +5V: now also VR1.3 (OUT)
- net GND: now also D8.2 (A2), VR1.2 (GND_2), VR1.4 (GND_4)
- new net: C1.1, C16.1, D8.1 (A1), F1.2, VR1.1 (IN)
Other:
- moved on the sheet: C15, C2, D2, H1, H2, H3, H4, R23
